Commit message: Added gait playground

File: awd/data/assets/mini_bdx/urdf/bdx.urdf (robot description, URDF)
Before this commit: robot bdx, 20 links, 19 joints
Links:
- link body_module: geometry visual mesh filename=../meshes/body_part.stl; visual mesh filename=../meshes/cage_back.stl
- link double_u_module: geometry visual mesh filename=../meshes/dc15_a01_horn_dummy.stl; visual mesh filename=../meshes/dc15_a01_horn_idle2_dummy.stl
- link double_u_module_2: geometry visual mesh filename=../meshes/dc15_a01_horn_dummy.stl; visual mesh filename=../meshes/dc15_a01_horn_dummy.stl
- link foot_module: geometry visual mesh filename=../meshes/dc15_a01_horn_dummy.stl; visual mesh filename=../meshes/dc15_a01_horn_idle2_dummy.stl
- link foot_module_2: geometry visual mesh filename=../meshes/dc15_a01_horn_dummy.stl; visual mesh filename=../meshes/dc15_a01_horn_idle2_dummy.stl
- link head_assembly: geometry visual mesh filename=../meshes/antenna_motor_holder.stl; visual mesh filename=../meshes/antenna_motor_holder.stl
- link head_link: geometry visual mesh filename=../meshes/axis_to_axis.stl; visual mesh filename=../meshes/axis_to_axis.stl
- link head_pitch_yaw: geometry visual mesh filename=../meshes/dc15_a01_case_b_dummy.stl; visual mesh filename=../meshes/dc15_a01_case_b_dummy.stl
- link left_antenna_assembly: geometry visual mesh filename=../meshes/antenna.stl; visual mesh filename=../meshes/antenna_holder_left.stl
- link left_hip_pitch_roll_module: geometry visual mesh filename=../meshes/dc15_a01_case_b_dummy.stl; visual mesh filename=../meshes/dc15_a01_case_b_dummy.stl
- link leg_module: geometry visual mesh filename=../meshes/block_to_axis.stl; visual mesh filename=../meshes/block_to_axis.stl
- link leg_module_2: geometry visual mesh filename=../meshes/block_to_axis.stl; visual mesh filename=../meshes/block_to_axis.stl
- link leg_module_3: geometry visual mesh filename=../meshes/block_to_axis.stl; visual mesh filename=../meshes/block_to_axis.stl
- link leg_module_4: geometry visual mesh filename=../meshes/block_to_axis.stl; visual mesh filename=../meshes/block_to_axis.stl
- link right_antenna_assembly: geometry visual mesh filename=../meshes/antenna.stl; visual mesh filename=../meshes/antenna_holder_right.stl
- link right_hip_pitch_roll_module: geometry visual mesh filename=../meshes/dc15_a01_case_b_dummy.stl; visual mesh filename=../meshes/dc15_a01_case_b_dummy.stl
